Commit message: add move_platform2

File: src/aimm_description/urdf/aimm.xacro (robot description, xacro)
@@ -50,8 +50,8 @@
 	</visual>
   </link>
-  <link name="kinect_supp1">
+  <link name="camera_link_supp1">
 	<visual>
 		<geometry>
-			<box size="0.04 0.04 0.2"/>
+			<box size="0.04 0.04 0.4"/>
 		</geometry>
 		<origin xyz="0 0 0"/>
@@ -59,5 +59,5 @@
 	</visual>
   </link>
-  <link name="kinect_supp2">
+  <link name="camera_link_supp2">
 	<visual>
 		<geometry>
@@ -68,5 +68,5 @@
 	</visual>
   </link>
-  <link name="kinect">
+  <link name="camera_link">
 	<visual>
 		<geometry>
@@ -75,18 +75,18 @@
 	</visual>
   </link>
-  <joint name="ur_base_link_to_kinect" type="fixed">
+  <joint name="ur_base_link_to_camera_link" type="fixed">
 	<parent link="ur_base_link"/>
-	<child link="kinect"/>
-	<origin xyz="-0.3541575 0.1507695 0.779517" rpy="-0.369 0.825 1.119"/>
+	<child link="camera_link"/>
+	<origin xyz="-0.547092 0.112523 0.586811" rpy="-0.219 0.636 1.266"/>
   </joint>
-  <joint name="supporter_to_kinect_supp1" type="fixed">
+  <joint name="supporter_to_camera_link_supp1" type="fixed">
 	<parent link="supporter"/>
-	<child link="kinect_supp1"/>
-	<origin xyz="0.03 0.15 0.44" rpy="1.57 0 0"/>
+	<child link="camera_link_supp1"/>
+	<origin xyz="0.03 0.25 0.44" rpy="1.57 0 0"/>
   </joint>
-  <joint name="supporter_to_kinect_supp2" type="fixed">
+  <joint name="supporter_to_camera_link_supp2" type="fixed">
 	<parent link="supporter"/>
-	<child link="kinect_supp2"/>
-	<origin xyz="0.03 0.27 0.87" rpy="0 0 0"/>
+	<child link="camera_link_supp2"/>
+	<origin xyz="0.03 0.47 0.87" rpy="0 0 0"/>
   </joint>
   <joint name="base_link_to_laser" type="fixed">
